File: model/popeye/popeye_model.sch (KiCad schematic (older format))
At the start: 18 parts, among them U1 74LS04, U1B1 74LS00, U1D1 74LS00, U1E1 74LS138, U1F1 74LS161, U1L1 74LS74, U2 74LS74, U2D 74LS74, U2E1 74LS161, U2F1 74LS161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

Commit message: minor
Parts:
- renumbered U2D to U2D1
Connections:
- net labels added: AI, BI, VB
Changed lines of the file:
@@
 $EndComp
 $Comp
-L 74LS74 U2D
+L 74LS74 U2D1
 U 1 1 5CFF7678
 P 2100 2600
-F 0 "U2D" H 2250 2900 50  0000 C CNN
+F 0 "U2D1" H 2250 2900 50  0000 C CNN
 F 1 "74LS74" H 2400 2305 50  0000 C CNN
 F 2 "" H 2100 2600 50  0000 C CNN
@@
 $EndComp
 $Comp
-L 74LS74 U2D
+L 74LS74 U2D1
 U 2 1 5CFF76D5
 P 3950 2600
-F 0 "U2D" H 4100 2900 50  0000 C CNN
+F 0 "U2D1" H 4100 2900 50  0000 C CNN
 F 1 "74LS74" H 4250 2305 50  0000 C CNN
 F 2 "" H 3950 2600 50  0000 C CNN
@@
 Text Label 3350 2400 2    60   ~ 0
 BUSAK
+Text Label 2150 6100 2    60   ~ 0
+BI
+Text Label 2400 7600 2    60   ~ 0
+AI
+Text Label 4200 8400 2    60   ~ 0
+VB
 $EndSCHEMATC
