File: model/popeye/dmasch.sch (KiCad schematic (older format))
At the start: 26 parts, among them U1 74LS04, U1B1 74LS00, U1D1 74LS00, U1E1 74LS138, U1F1 74LS161, U1L1 74LS74, U2 74LS74, U2D1 74LS74, U2E1 74LS161, U2F1 74LS161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

Commit message: minor
Parts:
- added pu19: rpullup, symbol arcade:rpullup
Connections:
- net DMCSpullup: now also pu19.1 (x)
- net DMclr_n: now also U3.11; no longer U3.3
- net at U1D1.3, U2.2 (D): now also U3.12; no longer U3.1
- net at U2.6 (~Q): now also U3.13; no longer U3.2
