File: model/popeye/dmasch.sch (KiCad schematic (older format))
At the start: 27 parts, among them U1 74LS04, U1B1 74LS00, U1D1 74LS00, U1E1 74LS138, U1F1 74LS161, U1L1 74LS74, U2 74LS74, U2D1 74LS74, U2E1 74LS161, U2F1 74LS161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

Commit message: wip
Parts:
- 1R1: simfile (none) -> \"dma21.bin\"
- 1S1: simfile (none) -> \"dma11.bin\"
- 1T1: simfile (none) -> \"dma01.bin\"
- 1U1: simfile (none) -> \"dma31.bin\"
- 2R1: simfile (none) -> \"dma20.bin\"
- 2S1: simfile (none) -> \"dma10.bin\"
- 2T1: simfile (none) -> \"dma00.bin\"
- 2U1: simfile (none) -> \"dma30.bin\"
Changed lines of the file:
@@
 F 2 "" H 18150 9100 50  0001 C CNN
 F 3 "" H 18150 9100 50  0001 C CNN
+F 4 "\"dma00.bin\"" H 18700 8800 50  0001 C CNN "simfile"
 	1    18700 8800
 	1    0    0    -1
@@
 F 2 "" H 18150 10600 50  0001 C CNN
 F 3 "" H 18150 10600 50  0001 C CNN
+F 4 "\"dma01.bin\"" H 18700 10300 50  0001 C CNN "simfile"
 	1    18700 10300
 	1    0    0    -1
@@
 F 2 "" H 20700 9100 50  0001 C CNN
 F 3 "" H 20700 9100 50  0001 C CNN
+F 4 "\"dma10.bin\"" H 21250 8800 50  0001 C CNN "simfile"
 	1    21250 8800
 	1    0    0    -1
@@
 F 2 "" H 20700 10600 50  0001 C CNN
 F 3 "" H 20700 10600 50  0001 C CNN
+F 4 "\"dma11.bin\"" H 21250 10300 50  0001 C CNN "simfile"
 	1    21250 10300
 	1    0    0    -1
@@
 F 2 "" H 18150 12050 50  0001 C CNN
 F 3 "" H 18150 12050 50  0001 C CNN
+F 4 "\"dma20.bin\"" H 18700 11750 50  0001 C CNN "simfile"
 	1    18700 11750
 	1    0    0    -1
@@
 F 2 "" H 18150 13550 50  0001 C CNN
 F 3 "" H 18150 13550 50  0001 C CNN
+F 4 "\"dma21.bin\"" H 18700 13250 50  0001 C CNN "simfile"
 	1    18700 13250
 	1    0    0    -1
@@
 F 2 "" H 20700 12050 50  0001 C CNN
 F 3 "" H 20700 12050 50  0001 C CNN
+F 4 "\"dma30.bin\"" H 21250 11750 50  0001 C CNN "simfile"
 	1    21250 11750
 	1    0    0    -1
@@
 F 2 "" H 20700 13550 50  0001 C CNN
 F 3 "" H 20700 13550 50  0001 C CNN
+F 4 "\"dma31.bin\"" H 21250 13250 50  0001 C CNN "simfile"
 	1    21250 13250
 	1    0    0    -1
