File: model/popeye/video1.sch (KiCad schematic (older format))
At the start: 39 parts, among them U3R1 74LS283, U3S1 74LS283, U3T1 74LS283, U5 74LS174, U6 74LS174, U7 74LS174

Commit message: wip
Parts:
- pu1, pu2, pu3, pu4, pu5, pu6, pu7, pu8, pu9: value pullup -> rpullup
Connections:
- net ADR0[3]: now reaches 1M2.1 (A[3]), 3M2.1 (A[3]), 4M1.12 (Zc)
- net ADR0[4]: now reaches 1M2.2 (A[4]), 3M2.2 (A[4]), 4N1.4 (Za)
- net ADR0[0]: now reaches 1M2.25 (A[0]), 3M2.25 (A[0]), 4M1.4 (Za)
- net ADR0[1]: now reaches 1M2.26 (A[1]), 3M2.26 (A[1]), 4M1.7 (Zb)
- net ADR0[2]: now reaches 1M2.27 (A[2]), 3M2.27 (A[2]), 4M1.9 (Zd)
- net ADR0[5]: now reaches 1M2.3 (A[5]), 3M2.3 (A[5]), 4N1.7 (Zb)
Other:
- moved on the sheet: 4B1B
Changed lines of the file:
@@
 $Descr A2 23386 16535
 encoding utf-8
-Sheet 3 3
+Sheet 3 4
 Title ""
 Date ""
@@
 Wire Wire Line
 	3150 2550 2450 2550
-Text HLabel 2450 2150 0    50   Input ~ 0
-ROHVS
-Text HLabel 2450 3200 0    50   Input ~ 0
-RVn
-Text HLabel 2450 2550 0    50   Input ~ 0
-ROHVCK
 Wire Wire Line
 	10000 5000 10000 2150
@@
 L jt74xx:74LS74 4B1
 U 2 1 5D464466
-P 4950 9450
-F 0 "4B1" H 5050 9700 50  0000 C CNN
-F 1 "74LS74" H 5000 9450 50  0000 C CNN
-F 2 "" H 4950 9450 50  0001 C CNN
-F 3 "74xx/74hc_hct74.pdf" H 4950 9450 50  0001 C CNN
-	2    4950 9450
-	1    0    0    -1
-$EndComp
-Wire Wire Line
-	5250 9550 5500 9550
-Text HLabel 5500 9550 2    50   Output ~ 0
-TXTCL
-NoConn ~ 5250 9350
-Wire Wire Line
-	4950 9150 4950 9050
-Wire Wire Line
-	4950 9050 5400 9050
-Wire Wire Line
-	5400 9050 5400 9750
-Wire Wire Line
-	5400 9750 4950 9750
-Text Label 4250 7750 2    50   ~ 0
-VDD
+P 4750 9450
+F 0 "4B1" H 4850 9700 50  0000 C CNN
+F 1 "74LS74" H 4800 9450 50  0000 C CNN
+F 2 "" H 4750 9450 50  0001 C CNN
+F 3 "74xx/74hc_hct74.pdf" H 4750 9450 50  0001 C CNN
+	2    4750 9450
+	1    0    0    -1
+$EndComp
+Wire Wire Line
+	5050 9550 5300 9550
+NoConn ~ 5050 9350
+Wire Wire Line
+	4750 9150 4750 9050
+Wire Wire Line
+	4750 9050 5200 9050
+Wire Wire Line
+	5200 9050 5200 9750
+Wire Wire Line
+	5200 9750 4750 9750
 $Comp
 L jt74xx:74LS74 4B1
@@
 	4400 8400 4400 9350
 Wire Wire Line
-	4400 9350 4650 9350
-Wire Wire Line
 	2000 7000 2350 7000
 Wire Wire Line
-	4650 9450 2350 9450
+	4450 9450 2350 9450
 Wire Wire Line
 	2350 9450 2350 7000
@@
 Wire Wire Line
 	2850 7800 2500 7800
-Text Label 5150 9050 0    50   ~ 0
+Text Label 4950 9050 0    50   ~ 0
 VDD
 $Comp
@@
 Text Label 7300 7950 2    50   ~ 0
 V[0]
-Text HLabel 7400 7000 0    50   Input ~ 0
-H2O
 Wire Wire Line
 	8200 7000 7650 7000
@@
 	7150 10850 8200 10850
 Connection ~ 7150 9400
-Text HLabel 7400 7500 0    50   Input ~ 0
-DO[2]
-Text HLabel 7400 7600 0    50   Input ~ 0
-DO[3]
-Text HLabel 7400 7700 0    50   Input ~ 0
-DO[4]
-Text HLabel 7400 7800 0    50   Input ~ 0
-DO[5]
 Wire Wire Line
 	8200 7500 8050 7500
@@
 Wire Wire Line
 	7400 7800 7900 7800
-Text HLabel 7400 8650 0    50   Input ~ 0
-DO[6]
-Text HLabel 7400 8750 0    50   Input ~ 0
-DO[7]
 Wire Wire Line
 	8200 8650 7800 8650
@@
 Text GLabel 9100 3150 2    50   Output ~ 0
 ROVI[8]
+Wire Wire Line
+	16650 2500 16650 3450
+Wire Wire Line
+	16650 3450 16600 3450
+Wire Wire Line
+	16750 2850 16750 3550
+Wire Wire Line
+	16750 3550 16600 3550
+Wire Wire Line
+	16850 2500 16850 3650
+Wire Wire Line
+	16850 3650 16600 3650
+Wire Wire Line
+	17000 2850 17000 3750
+Wire Wire Line
+	17000 3750 16600 3750
+Wire Wire Line
+	17100 2500 17100 3850
+Wire Wire Line
+	17100 3850 16600 3850
+Wire Wire Line
+	17200 2850 17200 3950
+Wire Wire Line
+	17200 3950 16600 3950
+Wire Wire Line
+	17300 2500 17300 4050
+Wire Wire Line
+	17300 4050 16600 4050
+Wire Wire Line
+	17450 2850 17450 4150
+Wire Wire Line
+	17450 4150 16600 4150
+Wire Wire Line
+	17550 2500 17550 4250
+Wire Wire Line
+	17550 4250 16600 4250
 $Comp
 L arcade:rpullup pu1
-U 1 1 5D805C82
+U 1 1 5DA333B0
 P 16650 2500
-F 0 "pu1" H 16600 3050 50  0000 L CNN
-F 1 "pullup" V 16550 2750 50  0000 L CNN
+F 0 "pu1" H 16728 2790 50  0000 L CNN
+F 1 "rpullup" H 16728 2699 50  0000 L CNN
 F 2 "" H 16450 2500 50  0001 C CNN
 F 3 "" H 16450 2500 50  0001 C CNN
@@
 $Comp
 L arcade:rpullup pu2
-U 1 1 5D805F3F
+U 1 1 5DA3345E
 P 16750 2850
-F 0 "pu2" H 16700 3400 50  0000 L CNN
-F 1 "pullup" V 16650 3100 50  0000 L CNN
+F 0 "pu2" H 16828 3140 50  0000 L CNN
+F 1 "rpullup" H 16828 3049 50  0000 L CNN
 F 2 "" H 16550 2850 50  0001 C CNN
 F 3 "" H 16550 2850 50  0001 C CNN
@@
 $Comp
 L arcade:rpullup pu3
-U 1 1 5D805FB9
+U 1 1 5DA3358D
 P 16850 2500
-F 0 "pu3" H 16800 3050 50  0000 L CNN
-F 1 "pullup" V 16750 2750 50  0000 L CNN
+F 0 "pu3" H 16928 2790 50  0000 L CNN
+F 1 "rpullup" H 16928 2699 50  0000 L CNN
 F 2 "" H 16650 2500 50  0001 C CNN
 F 3 "" H 16650 2500 50  0001 C CNN
@@
 $Comp
 L arcade:rpullup pu4
-U 1 1 5D806039
+U 1 1 5DA3361B
 P 17000 2850
-F 0 "pu4" H 16950 3400 50  0000 L CNN
-F 1 "pullup" V 16900 3100 50  0000 L CNN
+F 0 "pu4" H 17078 3140 50  0000 L CNN
+F 1 "rpullup" H 17078 3049 50  0000 L CNN
 F 2 "" H 16800 2850 50  0001 C CNN
 F 3 "" H 16800 2850 50  0001 C CNN
@@
 $Comp
 L arcade:rpullup pu5
-U 1 1 5D858217
+U 1 1 5DA336A7
 P 17100 2500
-F 0 "pu5" H 17050 3050 50  0000 L CNN
-F 1 "pullup" V 17000 2750 50  0000 L CNN
+F 0 "pu5" H 17178 2790 50  0000 L CNN
+F 1 "rpullup" H 17178 2699 50  0000 L CNN
 F 2 "" H 16900 2500 50  0001 C CNN
 F 3 "" H 16900 2500 50  0001 C CNN
@@
 $Comp
 L arcade:rpullup pu6
-U 1 1 5D85821E
+U 1 1 5DA337DF
 P 17200 2850
-F 0 "pu6" H 17150 3400 50  0000 L CNN
-F 1 "pullup" V 17100 3100 50  0000 L CNN
+F 0 "pu6" H 17278 3140 50  0000 L CNN
+F 1 "rpullup" H 17278 3049 50  0000 L CNN
 F 2 "" H 17000 2850 50  0001 C CNN
 F 3 "" H 17000 2850 50  0001 C CNN
@@
 $Comp
 L arcade:rpullup pu7
-U 1 1 5D858225
+U 1 1 5DA3386B
 P 17300 2500
-F 0 "pu7" H 17250 3050 50  0000 L CNN
-F 1 "pullup" V 17200 2750 50  0000 L CNN
+F 0 "pu7" H 17378 2790 50  0000 L CNN
+F 1 "rpullup" H 17378 2699 50  0000 L CNN
 F 2 "" H 17100 2500 50  0001 C CNN
 F 3 "" H 17100 2500 50  0001 C CNN
@@
 $Comp
 L arcade:rpullup pu8
-U 1 1 5D85822C
+U 1 1 5DA338F7
 P 17450 2850
-F 0 "pu8" H 17400 3400 50  0000 L CNN
-F 1 "pullup" V 17350 3100 50  0000 L CNN
+F 0 "pu8" H 17528 3140 50  0000 L CNN
+F 1 "rpullup" H 17528 3049 50  0000 L CNN
 F 2 "" H 17250 2850 50  0001 C CNN
 F 3 "" H 17250 2850 50  0001 C CNN
@@
 $Comp
 L arcade:rpullup pu9
-U 1 1 5D873464
+U 1 1 5DA33989
 P 17550 2500
-F 0 "pu9" H 17500 3050 50  0000 L CNN
-F 1 "pullup" V 17450 2750 50  0000 L CNN
+F 0 "pu9" H 17628 2790 50  0000 L CNN
+F 1 "rpullup" H 17628 2699 50  0000 L CNN
 F 2 "" H 17350 2500 50  0001 C CNN
 F 3 "" H 17350 2500 50  0001 C CNN
@@
 	1    0    0    -1
 $EndComp
-Wire Wire Line
-	16650 2500 16650 3450
-Wire Wire Line
-	16650 3450 16600 3450
-Wire Wire Line
-	16750 2850 16750 3550
-Wire Wire Line
-	16750 3550 16600 3550
-Wire Wire Line
-	16850 2500 16850 3650
-Wire Wire Line
-	16850 3650 16600 3650
-Wire Wire Line
-	17000 2850 17000 3750
-Wire Wire Line
-	17000 3750 16600 3750
-Wire Wire Line
-	17100 2500 17100 3850
-Wire Wire Line
-	17100 3850 16600 3850
-Wire Wire Line
-	17200 2850 17200 3950
-Wire Wire Line
-	17200 3950 16600 3950
-Wire Wire Line
-	17300 2500 17300 4050
-Wire Wire Line
-	17300 4050 16600 4050
-Wire Wire Line
-	17450 2850 17450 4150
-Wire Wire Line
-	17450 4150 16600 4150
-Wire Wire Line
-	17550 2500 17550 4250
-Wire Wire Line
-	17550 4250 16600 4250
+Text GLabel 7400 7000 0    50   Input ~ 0
+H2O
+Text GLabel 7400 7800 0    50   Input ~ 0
+DO[5]
+Text GLabel 7400 7700 0    50   Input ~ 0
+DO[4]
+Text GLabel 7400 7600 0    50   Input ~ 0
+DO[3]
+Text GLabel 7400 7500 0    50   Input ~ 0
+DO[2]
+Text GLabel 7400 8750 0    50   Input ~ 0
+DO[7]
+Text GLabel 7400 8650 0    50   Input ~ 0
+DO[6]
+Text Label 9450 7250 0    50   ~ 0
+ADR0[0]
+Text Label 9450 7350 0    50   ~ 0
+ADR0[1]
+Text Label 9450 7450 0    50   ~ 0
+ADR0[2]
+Text Label 9450 7550 0    50   ~ 0
+ADR0[3]
+Text Label 9450 8700 0    50   ~ 0
+ADR0[4]
+Text Label 9450 8800 0    50   ~ 0
+ADR0[5]
+Text GLabel 2450 2150 0    50   Input ~ 0
+ROHVS
+Text GLabel 2450 2550 0    50   Input ~ 0
+ROHVCK
+Text GLabel 2450 3200 0    50   Input ~ 0
+RVn
+Text GLabel 5300 9550 2    50   Output ~ 0
+TXTCL
+Wire Wire Line
+	4400 9350 4450 9350
 $EndSCHEMATC

Commit message: wip
Parts:
- added pu10, pu11, pu12, pu13, pu14, pu15, pu16, pu17, pu18: rpullup, symbol arcade:rpullup
Connections:
- net DJI[0]: now also pu10.1 (x)
- net DJI[1]: now also pu11.1 (x)
- net DJI[2]: now also pu12.1 (x)
- net DJI[3]: now also pu13.1 (x)
- net DJI[4]: now also pu14.1 (x)
- net DJI[5]: now also pu15.1 (x)
- net DJI[6]: now also pu16.1 (x)
- net DJI[7]: now also pu17.1 (x)
- net DJI[8]: now also pu18.1 (x)
Changed lines of the file:
@@
 Wire Wire Line
 	4400 9350 4450 9350
+$Comp
+L arcade:rpullup pu10
+U 1 1 5DB34EC5
+P 15400 2500
+F 0 "pu10" H 15478 2790 50  0000 L CNN
+F 1 "rpullup" H 15478 2699 50  0000 L CNN
+F 2 "" H 15200 2500 50  0001 C CNN
+F 3 "" H 15200 2500 50  0001 C CNN
+	1    15400 2500
+	1    0    0    -1
+$EndComp
+$Comp
+L arcade:rpullup pu11
+U 1 1 5DB34ECC
+P 15500 2850
+F 0 "pu11" H 15578 3140 50  0000 L CNN
+F 1 "rpullup" H 15578 3049 50  0000 L CNN
+F 2 "" H 15300 2850 50  0001 C CNN
+F 3 "" H 15300 2850 50  0001 C CNN
+	1    15500 2850
+	1    0    0    -1
+$EndComp
+$Comp
+L arcade:rpullup pu12
+U 1 1 5DB34ED3
+P 15600 2500
+F 0 "pu12" H 15678 2790 50  0000 L CNN
+F 1 "rpullup" H 15678 2699 50  0000 L CNN
+F 2 "" H 15400 2500 50  0001 C CNN
+F 3 "" H 15400 2500 50  0001 C CNN
+	1    15600 2500
+	1    0    0    -1
+$EndComp
+$Comp
+L arcade:rpullup pu13
+U 1 1 5DB34EDA
+P 15750 2850
+F 0 "pu13" H 15828 3140 50  0000 L CNN
+F 1 "rpullup" H 15828 3049 50  0000 L CNN
+F 2 "" H 15550 2850 50  0001 C CNN
+F 3 "" H 15550 2850 50  0001 C CNN
+	1    15750 2850
+	1    0    0    -1
+$EndComp
+$Comp
+L arcade:rpullup pu14
+U 1 1 5DB34EE1
+P 15850 2500
+F 0 "pu14" H 15928 2790 50  0000 L CNN
+F 1 "rpullup" H 15928 2699 50  0000 L CNN
+F 2 "" H 15650 2500 50  0001 C CNN
+F 3 "" H 15650 2500 50  0001 C CNN
+	1    15850 2500
+	1    0    0    -1
+$EndComp
+$Comp
+L arcade:rpullup pu15
+U 1 1 5DB34EE8
+P 15950 2850
+F 0 "pu15" H 16028 3140 50  0000 L CNN
+F 1 "rpullup" H 16028 3049 50  0000 L CNN
+F 2 "" H 15750 2850 50  0001 C CNN
+F 3 "" H 15750 2850 50  0001 C CNN
+	1    15950 2850
+	1    0    0    -1
+$EndComp
+$Comp
+L arcade:rpullup pu16
+U 1 1 5DB34EEF
+P 16050 2500
+F 0 "pu16" H 16128 2790 50  0000 L CNN
+F 1 "rpullup" H 16128 2699 50  0000 L CNN
+F 2 "" H 15850 2500 50  0001 C CNN
+F 3 "" H 15850 2500 50  0001 C CNN
+	1    16050 2500
+	1    0    0    -1
+$EndComp
+$Comp
+L arcade:rpullup pu17
+U 1 1 5DB34EF6
+P 16200 2850
+F 0 "pu17" H 16278 3140 50  0000 L CNN
+F 1 "rpullup" H 16278 3049 50  0000 L CNN
+F 2 "" H 16000 2850 50  0001 C CNN
+F 3 "" H 16000 2850 50  0001 C CNN
+	1    16200 2850
+	1    0    0    -1
+$EndComp
+$Comp
+L arcade:rpullup pu18
+U 1 1 5DB34EFD
+P 16300 2500
+F 0 "pu18" H 16378 2790 50  0000 L CNN
+F 1 "rpullup" H 16378 2699 50  0000 L CNN
+F 2 "" H 16100 2500 50  0001 C CNN
+F 3 "" H 16100 2500 50  0001 C CNN
+	1    16300 2500
+	1    0    0    -1
+$EndComp
+Text Label 15400 2850 3    50   ~ 0
+DJI[0]
+Text Label 15500 2850 3    50   ~ 0
+DJI[1]
+Text Label 15600 2850 3    50   ~ 0
+DJI[2]
+Wire Wire Line
+	15600 2850 15600 2500
+Wire Wire Line
+	15400 2500 15400 2850
+Wire Wire Line
+	15850 2500 15850 2850
+Text Label 15750 2850 3    50   ~ 0
+DJI[3]
+Text Label 15850 2850 3    50   ~ 0
+DJI[4]
+Text Label 15950 2850 3    50   ~ 0
+DJI[5]
+Text Label 16050 2850 3    50   ~ 0
+DJI[6]
+Text Label 16200 2850 3    50   ~ 0
+DJI[7]
+Text Label 16300 2850 3    50   ~ 0
+DJI[8]
+Wire Wire Line
+	16300 2850 16300 2500
+Wire Wire Line
+	16050 2850 16050 2500
 $EndSCHEMATC

Commit message: Added more labels
Connections:
- net DJ_latch_clk: now reaches 4A1.8, U5.9 (Cp), U6.9 (Cp), U7.9 (Cp)
- net carry: now reaches 1D1.9, U3T1.9 (C4)
- net train: now reaches 1D1.10, 1D1.11
- net DJ_CEn: now reaches 1D1.8, 4P2.3 (I1a), 4P2.5 (I0b)
- net H0H0or: now reaches 1D1.12, 2C1.11
- net H1n: now reaches 4A1.11, 5A1.12
- net HBn: now reaches 3A1.2, 4A1.3, 5A1.6
- net H0H0n: now reaches 3A2.3, 4A1.5, 8L1.1
- net preWEx: now reaches 3A1.8, 4P2.11 (I0d), 4P2.13 (I1c)
- net preWEy: now reaches 4P2.10 (I1d), 4P2.14 (I0c), 8L6.2
Changed lines of the file:
@@
 EESchema Schematic File Version 4
+LIBS:arcade
+LIBS:jt74xx
 LIBS:popeye_model-cache
 EELAYER 26 0
@@
 Text Label 3700 7100 0    50   ~ 0
 H0ln
-Text Label 3900 11600 2    50   ~ 0
+Text Label 3750 11600 2    50   ~ 0
 H0ln
 Wire Wire Line
@@
 Wire Wire Line
 	16050 2850 16050 2500
+Text Label 17700 4850 1    50   ~ 0
+DJ_latch_clk
+Text Label 7900 13200 0    50   ~ 0
+DJ_CEn
+Text Label 5550 6550 0    50   ~ 0
+H0H0n
+Text Label 4500 8700 0    50   ~ 0
+HBn
+Text Label 6750 11500 0    50   ~ 0
+preWEx
+Text Label 6750 12000 0    50   ~ 0
+preWEy
+Wire Wire Line
+	3900 11600 3750 11600
+Text Label 4500 12300 0    50   ~ 0
+H0H0or
+Text Label 9500 5550 0    50   ~ 0
+carry
+Text Label 10100 5700 0    50   ~ 0
+train
+Text Label 3800 7300 0    50   ~ 0
+H1n
 $EndSCHEMATC

Commit message: wip
Parts:
- renumbered 1M1 to 1P, 3M1 to 3P
Connections:
- net ADR1[0]: now also 1P.25 (A[0]), 3P.25 (A[0])
- net ADR1[1]: now also 1P.26 (A[1]), 3P.26 (A[1])
- net ADR1[2]: now also 1P.27 (A[2]), 3P.27 (A[2])
- net ADR1[3]: now also 1P.1 (A[3]), 3P.1 (A[3])
- net ADR1[4]: now also 1P.2 (A[4]), 3P.2 (A[4])
- net ADR1[5]: now also 1P.3 (A[5]), 3P.3 (A[5])
Changed lines of the file:
@@
 H[7]
 $Comp
-L arcade:RAM_7063 1M1
+L arcade:RAM_7063 1P
 U 1 1 5D683DBA
 P 13850 11400
-F 0 "1M1" H 13850 12165 50  0000 C CNN
+F 0 "1P" H 13850 12165 50  0000 C CNN
 F 1 "RAM_7063" H 13850 12074 50  0000 C CNN
 F 2 "" H 13850 11400 50  0001 C CNN
@@
 $EndComp
 $Comp
-L arcade:RAM_7063 3M1
+L arcade:RAM_7063 3P
 U 1 1 5D683DC1
 P 15850 11400
-F 0 "3M1" H 15850 12165 50  0000 C CNN
+F 0 "3P" H 15850 12165 50  0000 C CNN
 F 1 "RAM_7063" H 15850 12074 50  0000 C CNN
 F 2 "" H 15850 11400 50  0001 C CNN
@@
 Text Label 3800 7300 0    50   ~ 0
 H1n
+Wire Wire Line
+	13700 12150 13700 12700
+Wire Wire Line
+	13700 12700 15700 12700
+Wire Wire Line
+	15700 12700 15700 12150
+Wire Wire Line
+	13800 12150 13800 12600
+Wire Wire Line
+	13800 12600 15800 12600
+Wire Wire Line
+	15800 12600 15800 12150
+Wire Wire Line
+	13900 12150 13900 12500
+Wire Wire Line
+	13900 12500 15900 12500
+Wire Wire Line
+	15900 12500 15900 12150
+Wire Wire Line
+	14000 12150 14000 12400
+Wire Wire Line
+	14000 12400 16000 12400
+Wire Wire Line
+	16000 12400 16000 12150
+Wire Wire Line
+	14100 12150 14100 12300
+Wire Wire Line
+	14100 12300 16100 12300
+Wire Wire Line
+	16100 12300 16100 12150
+Wire Wire Line
+	14200 12150 14200 12200
+Wire Wire Line
+	14200 12200 16200 12200
+Wire Wire Line
+	16200 12200 16200 12150
+Text Label 13850 12700 0    50   ~ 0
+ADR1[5]
+Text Label 13850 12600 0    50   ~ 0
+ADR1[4]
+Text Label 14050 12500 0    50   ~ 0
+ADR1[3]
+Text Label 14050 12400 0    50   ~ 0
+ADR1[2]
+Text Label 14400 12300 0    50   ~ 0
+ADR1[1]
+Text Label 14400 12200 0    50   ~ 0
+ADR1[0]
 $EndSCHEMATC

Commit message: wip
Parts:
- renumbered U5 to 1L2, 1P to 1P1, U6 to 2L1, U7 to 3L1, 3P to 3P1
Connections:
- net v_halfcarry: now reaches U3R1.7 (C0), U3S1.9 (C4)
- net TXT_SHIFTn: now reaches 3A1.3, 4B1.12 (D)
Other:
- moved on the sheet: 3A1A
Changed lines of the file:
@@
 $Descr A2 23386 16535
 encoding utf-8
-Sheet 3 4
+Sheet 3 5
 Title ""
 Date ""
@@
 L jt74xx:74LS00 3A1
 U 1 1 5D4886B9
-P 4100 8400
-F 0 "3A1" H 4100 8400 50  0000 C CNN
-F 1 "74LS00" H 4100 8639 50  0000 C CNN
-F 2 "" H 4100 8400 50  0001 C CNN
-F 3 "http://www.ti.com/lit/gpn/sn74ls00" H 4100 8400 50  0001 C CNN
-	1    4100 8400
-	1    0    0    -1
-$EndComp
-Wire Wire Line
-	3200 8700 3800 8700
-Wire Wire Line
-	3800 8500 3800 8700
-Connection ~ 3800 8700
-Wire Wire Line
-	3800 8700 4750 8700
-Wire Wire Line
-	3250 8300 3800 8300
-Wire Wire Line
-	4400 8400 4400 9350
+P 3850 8400
+F 0 "3A1" H 3850 8400 50  0000 C CNN
+F 1 "74LS00" H 3850 8639 50  0000 C CNN
+F 2 "" H 3850 8400 50  0001 C CNN
+F 3 "http://www.ti.com/lit/gpn/sn74ls00" H 3850 8400 50  0001 C CNN
+	1    3850 8400
+	1    0    0    -1
+$EndComp
+Wire Wire Line
+	3550 8500 3550 8700
+Wire Wire Line
+	4150 8400 4150 9350
 Wire Wire Line
 	2000 7000 2350 7000
@@
 Connection ~ 15900 5350
 $Comp
-L jt74xx:74LS174 U5
+L jt74xx:74LS174 1L2
 U 1 1 5D424ED8
 P 18600 3800
-F 0 "U5" H 18800 3300 50  0000 C CNN
+F 0 "1L2" H 18800 3300 50  0000 C CNN
 F 1 "74LS174" H 18600 3600 50  0000 C CNN
 F 2 "" H 18600 3800 50  0001 C CNN
@@
 $EndComp
 $Comp
-L jt74xx:74LS174 U6
+L jt74xx:74LS174 2L1
 U 1 1 5D42510A
 P 18600 5000
-F 0 "U6" H 18800 4500 50  0000 C CNN
+F 0 "2L1" H 18800 4500 50  0000 C CNN
 F 1 "74LS174" H 18600 4800 50  0000 C CNN
 F 2 "" H 18600 5000 50  0001 C CNN
@@
 $EndComp
 $Comp
-L jt74xx:74LS174 U7
+L jt74xx:74LS174 3L1
 U 1 1 5D42519C
 P 18600 6200
-F 0 "U7" H 18800 5700 50  0000 C CNN
+F 0 "3L1" H 18800 5700 50  0000 C CNN
 F 1 "74LS174" H 18600 6000 50  0000 C CNN
 F 2 "" H 18600 6200 50  0001 C CNN
@@
 H[7]
 $Comp
-L arcade:RAM_7063 1P
+L arcade:RAM_7063 1P1
 U 1 1 5D683DBA
 P 13850 11400
-F 0 "1P" H 13850 12165 50  0000 C CNN
+F 0 "1P1" H 13850 12165 50  0000 C CNN
 F 1 "RAM_7063" H 13850 12074 50  0000 C CNN
 F 2 "" H 13850 11400 50  0001 C CNN
@@
 $EndComp
 $Comp
-L arcade:RAM_7063 3P
+L arcade:RAM_7063 3P1
 U 1 1 5D683DC1
 P 15850 11400
-F 0 "3P" H 15850 12165 50  0000 C CNN
+F 0 "3P1" H 15850 12165 50  0000 C CNN
 F 1 "RAM_7063" H 15850 12074 50  0000 C CNN
 F 2 "" H 15850 11400 50  0001 C CNN
@@
 Text GLabel 5300 9550 2    50   Output ~ 0
 TXTCL
-Wire Wire Line
-	4400 9350 4450 9350
 $Comp
 L arcade:rpullup pu10
@@
 Text Label 14400 12200 0    50   ~ 0
 ADR1[0]
+Text Label 7150 5050 0    50   ~ 0
+v_halfcarry
+Wire Wire Line
+	4150 8400 4250 8400
+Connection ~ 4150 8400
+Wire Wire Line
+	3200 8700 3550 8700
+Wire Wire Line
+	3250 8300 3550 8300
+Connection ~ 3550 8700
+Wire Wire Line
+	3550 8700 4750 8700
+Wire Wire Line
+	4150 9350 4450 9350
+Text GLabel 4250 8400 2    50   Output ~ 0
+TXT_SHIFTn
 $EndSCHEMATC
