File: model/popeye/video2.sch (KiCad schematic (older format))
At the start: 10 parts

Commit message: wip
Parts:
- added 1E2, 1F2: ROM_2764, symbol arcade:ROM_2764
- added 3C1: 74LS174, symbol jt74xx:74LS174
- added 3D1: 74LS10, symbol 74xx:74LS10
- added 3E2, 3F1: 74LS377, symbol jt74xx:74LS377
- added 4C1: 74LS175, symbol jt74xx:74LS175
- added 4D1: 74LS00, symbol jt74xx:74LS00
- added 4E2, 4F1, 4H1, 5F1: 74LS194, symbol jt74xx:74LS194
- added unit 4 of 5D1
- added unit 3 of 5D1
- added unit 1 of 5D1
- added 6C2: 74LS368, symbol jt74xx:74LS368
- added 6D1: 74LS367, symbol jt74xx:74LS367
- added 6E1, 7E1, 8H1, U2: 74LS161, symbol jt74xx:74LS161
- added 6F1, 7K1, 8C1: 74LS86, symbol jt74xx:74LS86
- added 7D1: 74LS04, symbol jt74xx:74LS04
- added 8B1: 74LS74, symbol jt74xx:74LS74
- added U1: 74LS10, symbol jt74xx:74LS10
- added pu20: rpullup, symbol arcade:rpullup
- 1J1: renamed from 1J; simfile 1J -> ../../rom/tpp2-v.1j
- 1K1: renamed from 1K; simfile 1k -> ../../rom/tpp2-v.1k
- gave numbers to parts that had none: 1
- renumbered 3K to 3K1, 4J to 4J1, 4K to 4K1, 4L to 4L1, 5D to 5D1, 5J to 5J1, 5K to 5K1
Connections:
- net DJEO: now also 1E2.10 (A0), 1F2.10 (A0)
- net DJ[10]: now also 1E2.21 (A10), 1F2.21 (A10)
- net DJ[16]: now also 1E2.2 (A12), 1F2.2 (A12), 3C1.6 (D2), U1.5
- net DJ[17]: now also 1E2.23 (A11), 1F2.23 (A11)
- net DJ[1]: now also 1E2.9 (A1), 1F2.9 (A1)
- net DJ[2]: now also 1E2.8 (A2), 1F2.8 (A2)
- net DJ[3]: now also 1E2.7 (A3), 1F2.7 (A3)
- net DJ[4]: now also 1E2.6 (A4), 1F2.6 (A4)
- net DJ[5]: now also 1E2.5 (A5), 1F2.5 (A5)
- net DJ[6]: now also 1E2.4 (A6), 1F2.4 (A6)
- net DJ[7]: now also 1E2.3 (A7), 1F2.3 (A7)
- net DJ[8]: now also 1E2.25 (A8), 1F2.25 (A8)
- net DJ[9]: now also 1E2.24 (A9), 1F2.24 (A9)
- net GND: now also 3C1.8 (GND)
- net S[0]: now also 4D1.11, 4E2.9 (S0), 4F1.9 (S0), 4H1.9 (S0), 5F1.9 (S0)
- net S[1]: now also 4D1.3, 4E2.10 (S1), 4F1.10 (S1), 4H1.10 (S1), 5F1.10 (S1)
- net VCC: now also 3C1.16 (VCC)
- net VDD: now also 1J1.27 (P), 1K1.27 (P), 1E2.27 (P), 1F2.27 (P), 3C1.1 (~Mr), 4C1.1 (~Mr), 4E2.1 (~CL), 4F1.1 (~CL), 4H1.1 (~CL), 5F1.1 (~CL), 6E1.1 (~MR), 6E1.10 (CET), 6E1.7 (CEP), 6E1.9 (~PE), 6F1.2, 7E1.1 (~MR), 7E1.10 (CET), 7E1.2 (CP), 7E1.9 (~PE), 8B1.1 (~R), 8B1.10 (~S), 8B1.13 (~R), 8B1.4 (~S), 8C1.1, 8C1.13, 8H1.1 (~MR), 8H1.7 (CEP), U2.10 (CET), U2.7 (CEP)
- net VSS: now also 1J1.20 (CEn), 1J1.22 (OEn), 1K1.20 (CEn), 1K1.22 (OEn), 1E2.20 (CEn), 1E2.22 (OEn), 1F2.20 (CEn), 1F2.22 (OEn), 3C1.13 (D4), 3C1.14 (D5), 3E2.1 (~E), 3F1.1 (~E), 4F1.7 (Dsl), 5F1.2 (Dsr), 6C2.1 (OEa), 6C2.15 (OEb), 6D1.1 (OEa), 6D1.15 (OEb), 8C1.4, 8H1.3 (D0), 8H1.4 (D1)
- net phi2: now reaches 4J1.11 (Cp), 4K1.11 (Cp), 4L1.11 (Cp), 5K1.11 (Cp)
- net phi2: now also 4E2.11 (Cp), 4F1.11 (Cp), 4H1.11 (Cp), 5F1.11 (Cp), 7D1.8
- net objv0_msb: now reaches 4K1.12 (Q3), 5J1.2 (I0a)
- net ROMclk: now reaches 3K1.11 (CP)
- net ROMclk: now also 3K2.11 (CP), 3E2.11 (CP), 3F1.11 (CP), 6D1.5 (O2a)
- net VB: now reaches 5J1.15 (E)
- net objv0_lsb: now reaches 5J1.3 (I1a), 5K1.15 (Q0)
- net objv1_msb: now reaches 5J1.5 (I0b)
- net objv1_msb: now also 4F1.12 (Q3)
- net objv1_lsb: now reaches 5J1.6 (I1b)
- net objv1_lsb: now also 5F1.15 (Q0)
- new net: 4F1.15 (Q0), 4H1.7 (Dsl)
- new net: 4F1.2 (Dsr), 4H1.12 (Q3)
- new net: 3F1.9 (Q3), 4F1.3 (P0)
- new net: 3F1.6 (Q2), 4F1.4 (P1)
- new net: 3F1.5 (Q1), 4F1.5 (P2)
- new net: 3F1.2 (Q0), 4F1.6 (P3)
- new net: 3F1.12 (Q4), 4H1.6 (P3)
- new net: 1F2.16 (Q4), 3F1.13 (D4)
- new net: 1F2.17 (Q5), 3F1.14 (D5)
- new net: 3F1.15 (Q5), 4H1.5 (P2)
- new net: 3F1.16 (Q6), 4H1.4 (P1)
- new net: 1F2.18 (Q6), 3F1.17 (D6)
- new net: 1F2.19 (Q7), 3F1.18 (D7)
- new net: 3F1.19 (Q7), 4H1.3 (P0)
- new net: 1F2.11 (Q0), 3F1.3 (D0)
- new net: 1F2.12 (Q1), 3F1.4 (D1)
- new net: 1F2.13 (Q2), 3F1.7 (D2)
- new net: 1F2.15 (Q3), 3F1.8 (D3)
- new net: 4E2.7 (Dsl), 4H1.15 (Q0)
- new net: 4E2.12 (Q3), 4H1.2 (Dsr)
- new net: 4E2.15 (Q0), 5F1.7 (Dsl)
- new net: 4E2.2 (Dsr), 5F1.12 (Q3)
- new net: 3E2.9 (Q3), 4E2.3 (P0)
- new net: 3E2.6 (Q2), 4E2.4 (P1)
- new net: 3E2.5 (Q1), 4E2.5 (P2)
- new net: 3E2.2 (Q0), 4E2.6 (P3)
- new net: 3E2.12 (Q4), 5F1.6 (P3)
- new net: 1E2.16 (Q4), 3E2.13 (D4)
- new net: 1E2.17 (Q5), 3E2.14 (D5)
- new net: 3E2.15 (Q5), 5F1.5 (P2)
- new net: 3E2.16 (Q6), 5F1.4 (P1)
- new net: 1E2.18 (Q6), 3E2.17 (D6)
- new net: 1E2.19 (Q7), 3E2.18 (D7)
- new net: 3E2.19 (Q7), 5F1.3 (P0)
- new net: 1E2.11 (Q0), 3E2.3 (D0)
- new net: 1E2.12 (Q1), 3E2.4 (D1)
- new net: 1E2.13 (Q2), 3E2.7 (D2)
- new net: 1E2.15 (Q3), 3E2.8 (D3)
- new net: 4D1.9, U2.15 (TC)
- new net: 3D1.9, 6C2.12 (I5), 6D1.6 (I3), 6E1.2 (CP), 7E1.13 (Q1), 8B1.11 (C), 8H1.2 (CP)
- new net: 7D1.11, 7E1.14 (Q0)
- new net: 7D1.10, 7D1.9
- new net: 3D1.10, 6D1.10 (I4), 6E1.14 (Q0)
- new net: 3D1.11, 6D1.12 (I5), 6E1.13 (Q1)
- new net: 6D1.14 (I6), 6E1.12 (Q2), 6F1.9
- new net: 3D1.8, 6D1.4 (I2)
- new net: 4D1.10, 6C2.2 (I1), 6D1.7 (O3a)
- new net: 6C2.3 (O1a), 6C2.4 (I2)
- new net: 6C2.5 (O2a), 6C2.6 (I3)
- new net: 4D1.13, 4D1.2, 4D1.4, 4D1.5, 4D1.8
- new net: 4C1.14 (~Q3), 4D1.12
- new net: 4C1.15 (Q3), 4D1.1
- new net: 4C1.9 (Cp), 4D1.6
- new net: 3C1.7 (Q2), 4C1.12 (D2)
- new net: 4C1.13 (D3), 5D1.3
- new net: 3C1.2 (Q0), 4C1.4 (D0)
- new net: 3C1.5 (Q1), 4C1.5 (D1)
- new net: 6E1.11 (Q3), 6F1.4
- new net: 6E1.15 (TC), 8H1.10 (CET)
- new net: 7K1.1, 8H1.11 (Q3)
- new net: 7K1.12, 8H1.12 (Q2)
- new net: 7K1.4, 8H1.13 (Q1)
- new net: 7K1.9, 8H1.14 (Q0)
- new net: 8C1.2, 8H1.15 (TC)
- new net: 8B1.12 (D), 8B1.5 (Q), 8H1.5 (D2), 8H1.6 (D3)
- new net: 8C1.12, 8C1.3
- new net: 8B1.3 (C), 8C1.11
- new net: 8B1.2 (D), 8B1.6 (~Q)
- new net CLK20: 7E1.7 (CEP)
- new net DJ[11]: 3C1.11 (D3)
- new net DJ[12]: 5D1.9
- new net DJ[13]: 5D1.12
- new net DJ[14]: 3C1.3 (D0), U1.3
- new net DJ[15]: 3C1.4 (D1), U1.4
- new net DOTCK: 6C2.7 (O3a)
- new net H2O: 6F1.8
- new net HB: 8B1.9 (Q)
- new net HBn: 8B1.8 (~Q)
- new net H[0]: 6D1.9 (O4a)
- new net H[1]: 6D1.11 (O5b)
- new net H[2]: 6D1.13 (O6b)
- new net H[3]: 6F1.6
- new net H[4]: 7K1.8
- new net H[5]: 7K1.6
- new net H[6]: 7K1.11
- new net H[7]: 7K1.3
- new net OBJC[0]: 4C1.3 (~Q0)
- new net OBJC[1]: 4C1.6 (~Q1)
- new net OBJC[2]: 4C1.11 (~Q2)
- new net RV: 5D1.10, 5D1.13, 5D1.2, 8C1.6
- new net RVn: 6F1.1
- new net RVx: 6F1.10, 6F1.3, 6F1.5, 7K1.10, 7K1.13, 7K1.2, 7K1.5, 8C1.5
- new net hflip: 3C1.10 (Q3), 5D1.1
- new net objcnt_clk: 6C2.11 (O5b), U2.2 (CP)
- new net objcnt_start[0]: 5D1.8, U2.3 (D0)
- new net objcnt_start[1]: 5D1.11, U2.4 (D1)
- new net objcnt_start[2]: U2.5 (D2), pu20.1 (x)
- new net objcnt_start[3]: U1.6, U2.6 (D3)
- no-connect marks 6 -> 26
Other:
- note added: "Horizontal Counter"
- moved on the sheet: 1J1, 1K1, 3K1, 3K2, 4J1, 4K1, 4L1, 5D1B, 5J1, 5K1

Commit message: Fixed H cnt
Connections:
- net CLK20: now also 7E1.2 (CP); no longer 7E1.7 (CEP)
- net VDD: now also 7E1.7 (CEP); no longer 7E1.2 (CP)
- net Hclk: now reaches 3D1.9, 6C2.12 (I5), 6D1.6 (I3), 6E1.2 (CP), 7E1.13 (Q1), 8B1.11 (C), 8H1.2 (CP)
- net Hcnt_rstn: now reaches 8H1.9 (~PE)
- net Hcnt_rstn: now also 8C1.12, 8C1.3
Changed lines of the file:
@@
 	1    0    0    -1
 $EndComp
-Text GLabel 8650 8750 0    50   Input ~ 0
+Text GLabel 8600 8950 0    50   Input ~ 0
 CLK20
 Wire Wire Line
-	8650 8750 8850 8750
-Wire Wire Line
 	8850 8650 8750 8650
 Wire Wire Line
-	8750 8650 8750 8850
+	8750 8650 8750 8750
 Wire Wire Line
 	8750 8850 8850 8850
-Wire Wire Line
-	8750 8850 8750 8950
-Wire Wire Line
-	8750 8950 8850 8950
 Connection ~ 8750 8850
 Text Label 8850 8650 2    50   ~ 0
 VDD
 Wire Wire Line
-	8750 8950 8750 9150
-Wire Wire Line
 	8750 9150 8850 9150
-Connection ~ 8750 8950
 NoConn ~ 9850 8650
 NoConn ~ 9850 8450
@@
 VDD
 Wire Wire Line
-	17200 10800 17350 10800
+	17200 10800 17250 10800
 $Comp
 L jt74xx:74LS74 8B1
@@
 Text Label 4000 2150 2    50   ~ 0
 ROMclk
+Wire Wire Line
+	8750 8850 8750 9150
+Wire Wire Line
+	8600 8950 8850 8950
+Wire Wire Line
+	8850 8750 8750 8750
+Connection ~ 8750 8750
+Wire Wire Line
+	8750 8750 8750 8850
+Wire Wire Line
+	17250 10800 17250 10050
+Wire Wire Line
+	17250 10050 13500 10050
+Wire Wire Line
+	13500 10050 13500 10700
+Wire Wire Line
+	13500 10700 13600 10700
+Connection ~ 17250 10800
+Wire Wire Line
+	17250 10800 17350 10800
+Text Label 16650 10050 2    50   ~ 0
+Hcnt_rstn
+Text Label 12350 9450 2    50   ~ 0
+Hclk
 $EndSCHEMATC

Commit message: wip
Parts:
- added 5C1: 74LS74, symbol jt74xx:74LS74
- added 6A1: 74LS04, symbol jt74xx:74LS04
- added unit 3 of 8C1
- added U3: delay, symbol arcade:delay
- 1E2: simfile ../../rom/tpp2-v.1e -> \"../../rom/tpp2-v.1e\"
- 1F2: simfile ../../rom/tpp2-v.1f -> \"../../rom/tpp2-v.1f\"
- 1J1: simfile ../../rom/tpp2-v.1j -> \"../../rom/tpp2-v.1j\"
- 1K1: simfile ../../rom/tpp2-v.1k -> \"../../rom/tpp2-v.1k\"
- renumbered 3K2 to 3J1
Connections:
- net HB: now also 5C1.2 (D)
- net INIT_EOn: now also 6A1.12
- net RV: now also 8C1.10
- net VB: now also 5C1.3 (C)
- net VDD: now also 5C1.1 (~R), 5C1.4 (~S)
- net objlatch[3]: now reaches 3K1.9 (Q3), 4K1.3 (P0)
- net objlatch[2]: now reaches 3K1.6 (Q2), 4K1.4 (P1)
- net objlatch[1]: now reaches 3K1.5 (Q1), 4K1.5 (P2)
- net objlatch[0]: now reaches 3K1.2 (Q0), 4K1.6 (P3)
- net objlatch[4]: now reaches 3K1.12 (Q4), 4L1.6 (P3)
- net objrom[4]: now reaches 1K1.16 (Q4), 3K1.13 (D4)
- net objrom[5]: now reaches 1K1.17 (Q5), 3K1.14 (D5)
- net objlatch[5]: now reaches 3K1.15 (Q5), 4L1.5 (P2)
- net objlatch[6]: now reaches 3K1.16 (Q6), 4L1.4 (P1)
- net objrom[6]: now reaches 1K1.18 (Q6), 3K1.17 (D6)
- net objrom[7]: now reaches 1K1.19 (Q7), 3K1.18 (D7)
- net objlatch[7]: now reaches 3K1.19 (Q7), 4L1.3 (P0)
- net objrom[0]: now reaches 1K1.11 (Q0), 3K1.3 (D0)
- net objrom[1]: now reaches 1K1.12 (Q1), 3K1.4 (D1)
- net objrom[2]: now reaches 1K1.13 (Q2), 3K1.7 (D2)
- net objrom[3]: now reaches 1K1.15 (Q3), 3K1.8 (D3)
- net objlatch[11]: now reaches 3J1.9 (Q3), 4J1.3 (P0)
- net objlatch[10]: now reaches 3J1.6 (Q2), 4J1.4 (P1)
- net objlatch[9]: now reaches 3J1.5 (Q1), 4J1.5 (P2)
- net objlatch[8]: now reaches 3J1.2 (Q0), 4J1.6 (P3)
- net objlatch[12]: now reaches 3J1.12 (Q4), 5K1.6 (P3)
- net objrom[12]: now reaches 1J1.16 (Q4), 3J1.13 (D4)
- net objrom[13]: now reaches 1J1.17 (Q5), 3J1.14 (D5)
- net objlatch[13]: now reaches 3J1.15 (Q5), 5K1.5 (P2)
- net objlatch[14]: now reaches 3J1.16 (Q6), 5K1.4 (P1)
- net objrom[14]: now reaches 1J1.18 (Q6), 3J1.17 (D6)
- net objrom[15]: now reaches 1J1.19 (Q7), 3J1.18 (D7)
- net objlatch[15]: now reaches 3J1.19 (Q7), 5K1.3 (P0)
- net objrom[8]: now reaches 1J1.11 (Q0), 3J1.3 (D0)
- net objrom[9]: now reaches 1J1.12 (Q1), 3J1.4 (D1)
- net objrom[10]: now reaches 1J1.13 (Q2), 3J1.7 (D2)
- net objrom[11]: now reaches 1J1.15 (Q3), 3J1.8 (D3)
- net objlatch[19]: now reaches 3F1.9 (Q3), 4F1.3 (P0)
- net objlatch[18]: now reaches 3F1.6 (Q2), 4F1.4 (P1)
- net objlatch[17]: now reaches 3F1.5 (Q1), 4F1.5 (P2)
- net objlatch[16]: now reaches 3F1.2 (Q0), 4F1.6 (P3)
- net objlatch[20]: now reaches 3F1.12 (Q4), 4H1.6 (P3)
- net objrom[20]: now reaches 1F2.16 (Q4), 3F1.13 (D4)
- net objrom[21]: now reaches 1F2.17 (Q5), 3F1.14 (D5)
- net objlatch[21]: now reaches 3F1.15 (Q5), 4H1.5 (P2)
- net objlatch[22]: now reaches 3F1.16 (Q6), 4H1.4 (P1)
- net objrom[22]: now reaches 1F2.18 (Q6), 3F1.17 (D6)
- net objrom[23]: now reaches 1F2.19 (Q7), 3F1.18 (D7)
- net objlatch[23]: now reaches 3F1.19 (Q7), 4H1.3 (P0)
- net objrom[16]: now reaches 1F2.11 (Q0), 3F1.3 (D0)
- net objrom[17]: now reaches 1F2.12 (Q1), 3F1.4 (D1)
- net objrom[18]: now reaches 1F2.13 (Q2), 3F1.7 (D2)
- net objrom[19]: now reaches 1F2.15 (Q3), 3F1.8 (D3)
- net objlatch[27]: now reaches 3E2.9 (Q3), 4E2.3 (P0)
- net objlatch[26]: now reaches 3E2.6 (Q2), 4E2.4 (P1)
- net objlatch[25]: now reaches 3E2.5 (Q1), 4E2.5 (P2)
- net objlatch[24]: now reaches 3E2.2 (Q0), 4E2.6 (P3)
- net objlatch[28]: now reaches 3E2.12 (Q4), 5F1.6 (P3)
- net objrom[28]: now reaches 1E2.16 (Q4), 3E2.13 (D4)
- net objrom[29]: now reaches 1E2.17 (Q5), 3E2.14 (D5)
- net objlatch[29]: now reaches 3E2.15 (Q5), 5F1.5 (P2)
- net objlatch[30]: now reaches 3E2.16 (Q6), 5F1.4 (P1)
- net objrom[30]: now reaches 1E2.18 (Q6), 3E2.17 (D6)
- net objrom[31]: now reaches 1E2.19 (Q7), 3E2.18 (D7)
- net objlatch[31]: now reaches 3E2.19 (Q7), 5F1.3 (P0)
- net objrom[24]: now reaches 1E2.11 (Q0), 3E2.3 (D0)
- net objrom[25]: now reaches 1E2.12 (Q1), 3E2.4 (D1)
- net objrom[26]: now reaches 1E2.13 (Q2), 3E2.7 (D2)
- net objrom[27]: now reaches 1E2.15 (Q3), 3E2.8 (D3)
- net ROMclk_base: now reaches 3D1.8
- net ROMclk_base: now also U3.1 (a); no longer 6D1.4 (I2)
- new net: 6A1.13, 8C1.8
- new net: 5C1.6 (~Q), 8C1.9
- new net ROMclk_filtered: 6D1.4 (I2), U3.2 (y)
- no-connect marks 26 -> 27
Changed lines of the file:
@@
 F 2 "" H 2950 1850 50  0001 C CNN
 F 3 "" H 2950 1850 50  0001 C CNN
-F 4 "../../rom/tpp2-v.1k" H 2950 1850 50  0001 C CNN "simfile"
+F 4 "\"../../rom/tpp2-v.1k\"" H 2950 1850 50  0001 C CNN "simfile"
 	1    2950 1850
 	1    0    0    -1
@@
 $EndComp
 $Comp
-L jt74xx:74LS377 3K2
+L jt74xx:74LS377 3J1
 U 1 1 5D12A882
 P 4500 4400
-F 0 "3K2" H 4500 4400 50  0000 C CNN
+F 0 "3J1" H 4500 4400 50  0000 C CNN
 F 1 "74LS377" H 4600 3900 50  0000 C CNN
 F 2 "" H 4500 4400 50  0001 C CNN
@@
 F 2 "" H 2950 4500 50  0001 C CNN
 F 3 "" H 2950 4500 50  0001 C CNN
-F 4 "../../rom/tpp2-v.1j" H 2950 4500 50  0001 C CNN "simfile"
+F 4 "\"../../rom/tpp2-v.1j\"" H 2950 4500 50  0001 C CNN "simfile"
 	1    2950 4500
 	1    0    0    -1
@@
 Wire Wire Line
 	1300 1150 1150 1150
-Text GLabel 1150 1150 0    50   Input ~ 0
-INIT_EOn
 Text GLabel 2350 2450 0    50   Input ~ 0
 DJ[16]
@@
 F 2 "" H 2950 7000 50  0001 C CNN
 F 3 "" H 2950 7000 50  0001 C CNN
-F 4 "../../rom/tpp2-v.1f" H 2950 7000 50  0001 C CNN "simfile"
+F 4 "\"../../rom/tpp2-v.1f\"" H 2950 7000 50  0001 C CNN "simfile"
 	1    2950 7000
 	1    0    0    -1
@@
 F 2 "" H 2950 9650 50  0001 C CNN
 F 3 "" H 2950 9650 50  0001 C CNN
-F 4 "../../rom/tpp2-v.1e" H 2950 9650 50  0001 C CNN "simfile"
+F 4 "\"../../rom/tpp2-v.1e\"" H 2950 9650 50  0001 C CNN "simfile"
 	1    2950 9650
 	1    0    0    -1
@@
 	12050 9850 12050 10000
 Wire Wire Line
-	10500 9950 10500 8400
+	10500 9950 10500 9400
 Wire Wire Line
 	10500 8400 12200 8400
@@
 Text Label 12350 9450 2    50   ~ 0
 Hclk
+Text Label 3550 1250 0    50   ~ 0
+objrom[0]
+Text Label 3550 1350 0    50   ~ 0
+objrom[1]
+Text Label 3550 1450 0    50   ~ 0
+objrom[2]
+Text Label 3550 1550 0    50   ~ 0
+objrom[3]
+Text Label 3550 1650 0    50   ~ 0
+objrom[4]
+Text Label 3550 1750 0    50   ~ 0
+objrom[5]
+Text Label 3550 1850 0    50   ~ 0
+objrom[6]
+Text Label 3550 1950 0    50   ~ 0
+objrom[7]
+Text Label 3550 3900 0    50   ~ 0
+objrom[8]
+Text Label 3550 4000 0    50   ~ 0
+objrom[9]
+Text Label 3550 4100 0    50   ~ 0
+objrom[10]
+Text Label 3550 4200 0    50   ~ 0
+objrom[11]
+Text Label 3550 4300 0    50   ~ 0
+objrom[12]
+Text Label 3550 4400 0    50   ~ 0
+objrom[13]
+Text Label 3550 4600 0    50   ~ 0
+objrom[15]
+Text Label 3550 6400 0    50   ~ 0
+objrom[16]
+Text Label 3550 6500 0    50   ~ 0
+objrom[17]
+Text Label 3550 6600 0    50   ~ 0
+objrom[18]
+Text Label 3550 6700 0    50   ~ 0
+objrom[19]
+Text Label 3550 6800 0    50   ~ 0
+objrom[20]
+Text Label 3550 6900 0    50   ~ 0
+objrom[21]
+Text Label 3550 7000 0    50   ~ 0
+objrom[22]
+Text Label 3550 7100 0    50   ~ 0
+objrom[23]
+Text Label 3550 9050 0    50   ~ 0
+objrom[24]
+Text Label 3550 9150 0    50   ~ 0
+objrom[25]
+Text Label 3550 9250 0    50   ~ 0
+objrom[26]
+Text Label 3550 9350 0    50   ~ 0
+objrom[27]
+Text Label 3550 9450 0    50   ~ 0
+objrom[28]
+Text Label 3550 9550 0    50   ~ 0
+objrom[29]
+Text Label 3550 9750 0    50   ~ 0
+objrom[31]
+Text Label 3550 9650 0    50   ~ 0
+objrom[30]
+Text Label 3550 4500 0    50   ~ 0
+objrom[14]
+Text Label 5000 1250 0    50   ~ 0
+objlatch[0]
+Text Label 5000 1350 0    50   ~ 0
+objlatch[1]
+Text Label 5000 1450 0    50   ~ 0
+objlatch[2]
+Text Label 5000 1550 0    50   ~ 0
+objlatch[3]
+Text Label 5000 1650 0    50   ~ 0
+objlatch[4]
+Text Label 5000 1750 0    50   ~ 0
+objlatch[5]
+Text Label 5000 1850 0    50   ~ 0
+objlatch[6]
+Text Label 5000 1950 0    50   ~ 0
+objlatch[7]
+Text Label 5000 3900 0    50   ~ 0
+objlatch[8]
+Text Label 5000 4000 0    50   ~ 0
+objlatch[9]
+Text Label 5000 4100 0    50   ~ 0
+objlatch[10]
+Text Label 5000 4200 0    50   ~ 0
+objlatch[11]
+Text Label 5000 4300 0    50   ~ 0
+objlatch[12]
+Text Label 5000 4400 0    50   ~ 0
+objlatch[13]
+Text Label 5000 4500 0    50   ~ 0
+objlatch[14]
+Text Label 5000 4600 0    50   ~ 0
+objlatch[15]
+Text Label 5000 6400 0    50   ~ 0
+objlatch[16]
+Text Label 5000 6500 0    50   ~ 0
+objlatch[17]
+Text Label 5000 6600 0    50   ~ 0
+objlatch[18]
+Text Label 5000 6700 0    50   ~ 0
+objlatch[19]
+Text Label 5000 6800 0    50   ~ 0
+objlatch[20]
+Text Label 5000 6900 0    50   ~ 0
+objlatch[21]
+Text Label 5000 7000 0    50   ~ 0
+objlatch[22]
+Text Label 5000 7100 0    50   ~ 0
+objlatch[23]
+Text Label 5000 9050 0    50   ~ 0
+objlatch[24]
+Text Label 5000 9150 0    50   ~ 0
+objlatch[25]
+Text Label 5000 9250 0    50   ~ 0
+objlatch[26]
+Text Label 5000 9350 0    50   ~ 0
+objlatch[27]
+Text Label 5000 9450 0    50   ~ 0
+objlatch[28]
+Text Label 5000 9550 0    50   ~ 0
+objlatch[29]
+Text Label 5000 9650 0    50   ~ 0
+objlatch[30]
+Text Label 5000 9750 0    50   ~ 0
+objlatch[31]
+$Comp
+L jt74xx:74LS04 6A1
+U 6 1 5D17AC8D
+P 20350 3950
+F 0 "6A1" H 20350 4267 50  0000 C CNN
+F 1 "74LS04" H 20350 4176 50  0000 C CNN
+F 2 "" H 20350 3950 50  0001 C CNN
+F 3 "http://www.ti.com/lit/gpn/sn74LS04" H 20350 3950 50  0001 C CNN
+	6    20350 3950
+	1    0    0    -1
+$EndComp
+Wire Wire Line
+	20650 3950 20800 3950
+Text Label 20800 3950 0    50   ~ 0
+INIT_EOn
+Text Label 1150 1150 2    50   ~ 0
+INIT_EOn
+$Comp
+L jt74xx:74LS86 8C1
+U 3 1 5D1BC1AA
+P 19650 3950
+F 0 "8C1" H 19650 3633 50  0000 C CNN
+F 1 "74LS86" H 19650 3724 50  0000 C CNN
+F 2 "" H 19650 3950 50  0001 C CNN
+F 3 "74xx/74ls86.pdf" H 19650 3950 50  0001 C CNN
+	3    19650 3950
+	1    0    0    1
+$EndComp
+Wire Wire Line
+	19950 3950 20050 3950
+$Comp
+L jt74xx:74LS74 5C1
+U 1 1 5D23E319
+P 18250 3950
+F 0 "5C1" H 18250 4428 50  0000 C CNN
+F 1 "74LS74" H 18250 4337 50  0000 C CNN
+F 2 "" H 18250 3950 50  0001 C CNN
+F 3 "74xx/74hc_hct74.pdf" H 18250 3950 50  0001 C CNN
+	1    18250 3950
+	1    0    0    -1
+$EndComp
+Wire Wire Line
+	18550 4050 19350 4050
+Wire Wire Line
+	19350 3850 19200 3850
+Text Label 19200 3850 0    50   ~ 0
+RV
+NoConn ~ 18550 3850
+Wire Wire Line
+	17950 3850 17800 3850
+Text Label 17800 3850 2    50   ~ 0
+HB
+Wire Wire Line
+	17950 3950 17800 3950
+Text GLabel 17800 3950 0    50   Input ~ 0
+VB
+Wire Wire Line
+	18250 3650 18700 3650
+Wire Wire Line
+	18700 3650 18700 4250
+Wire Wire Line
+	18700 4250 18250 4250
+Text Label 18250 4250 0    50   ~ 0
+VDD
+$Comp
+L arcade:delay U3
+U 1 1 5D3CB60D
+P 10500 9100
+F 0 "U3" V 10616 8922 50  0000 R CNN
+F 1 "delay" V 10525 8922 50  0000 R CNN
+F 2 "" H 10500 9100 50  0001 C CNN
+F 3 "" H 10500 9100 50  0001 C CNN
+F 4 "40" V 10434 8922 50  0000 R CNN "delay_time"
+	1    10500 9100
+	0    -1   -1   0
+$EndComp
+Wire Wire Line
+	10500 8750 10500 8400
+Text Label 10500 9900 1    50   ~ 0
+ROMclk_base
+Text Label 10500 8400 0    50   ~ 0
+ROMclk_filtered
 $EndSCHEMATC

Commit message: wip
Parts:
- renumbered U2 to 5E1
Connections:
- net ROMclk: now also 3C1.9 (Cp), 5E1.9 (~PE)
- net objcnt[3]: now reaches 5E1.11 (Q3)
- net objcnt[2]: now reaches 5E1.12 (Q2)
- net objcnt[1]: now reaches 5E1.13 (Q1)
- net objcnt[0]: now reaches 5E1.14 (Q0)
Changed lines of the file:
@@
 Connection ~ 9950 5450
 $Comp
-L jt74xx:74LS161 U2
+L jt74xx:74LS161 5E1
 U 1 1 5D2A7693
 P 12700 5850
-F 0 "U2" H 12700 5850 50  0000 C CNN
+F 0 "5E1" H 12700 5850 50  0000 C CNN
 F 1 "74LS161" H 12850 5350 50  0000 C CNN
 F 2 "" H 12700 5850 50  0001 C CNN
@@
 Wire Wire Line
 	13200 8400 13300 8400
-Wire Wire Line
-	13300 8400 13300 8150
 Wire Wire Line
 	4000 9950 3800 9950
@@
 Text Label 10500 8400 0    50   ~ 0
 ROMclk_filtered
+Wire Wire Line
+	12200 5850 11850 5850
+Wire Wire Line
+	11850 5850 11850 7950
+Wire Wire Line
+	11850 7950 13300 7950
+Wire Wire Line
+	13300 7950 13300 8400
+Wire Wire Line
+	12000 4100 11850 4100
+Wire Wire Line
+	11850 4100 11850 5850
+Connection ~ 11850 5850
+Wire Wire Line
+	13300 5350 13200 5350
+Wire Wire Line
+	13300 5450 13200 5450
+Wire Wire Line
+	13300 5550 13200 5550
+Wire Wire Line
+	13300 5650 13200 5650
+Text Label 13300 5650 0    50   ~ 0
+objcnt[3]
+Text Label 13300 5550 0    50   ~ 0
+objcnt[2]
+Text Label 13300 5450 0    50   ~ 0
+objcnt[1]
+Text Label 13300 5350 0    50   ~ 0
+objcnt[0]
 $EndSCHEMATC

Commit message: wip
Connections:
- net obj_carry: now reaches 4D1.9, 5E1.15 (TC)
Changed lines of the file:
@@
 $EndComp
 Wire Wire Line
-	13450 5850 13200 5850
+	13450 5850 13400 5850
 $Comp
 L jt74xx:74LS00 4D1
@@
 Text Label 13300 5350 0    50   ~ 0
 objcnt[0]
+Text Label 13400 5750 2    50   ~ 0
+obj_carry
+Wire Wire Line
+	13400 5750 13400 5850
+Connection ~ 13400 5850
+Wire Wire Line
+	13400 5850 13200 5850
 $EndSCHEMATC

Commit message: Object test
Parts:
- removed 3D1: 74LS10, symbol 74xx:74LS10
- added 3D: 74LS10, symbol jt74xx:74LS10
Connections:
- net Hclk: now also 3D.9
- net ROMclk_base: now also 3D.8
- net at 6D1.10 (I4), 6E1.14 (Q0): now also 3D.10
- net at 6D1.12 (I5), 6E1.13 (Q1): now also 3D.11
Changed lines of the file:
@@
 Text Label 2850 10550 3    50   ~ 0
 VSS
-$Comp
-L 74xx:74LS10 3D1
-U 3 1 5EAACC7A
-P 10800 9950
-F 0 "3D1" H 10800 9633 50  0000 C CNN
-F 1 "74LS10" H 10800 9724 50  0000 C CNN
-F 2 "" H 10800 9950 50  0001 C CNN
-F 3 "http://www.ti.com/lit/gpn/sn74LS10" H 10800 9950 50  0001 C CNN
-	3    10800 9950
-	-1   0    0    1
-$EndComp
 Wire Wire Line
 	11100 10050 11900 10050
@@
 Wire Wire Line
 	13400 5850 13200 5850
+$Comp
+L jt74xx:74LS10 3D
+U 3 1 5D2DE440
+P 10800 9950
+F 0 "3D" H 10800 9633 50  0000 C CNN
+F 1 "74LS10" H 10800 9724 50  0000 C CNN
+F 2 "" H 10800 9950 50  0001 C CNN
+F 3 "http://www.ti.com/lit/gpn/sn74LS10" H 10800 9950 50  0001 C CNN
+	3    10800 9950
+	-1   0    0    1
+$EndComp
 $EndSCHEMATC
